Commit message: Update measured wheel dimensions across all files
wheel_radius: 0.034 → 0.033 m (66 mm measured diameter)
wheel_separation: 0.179 → 0.177 m (measured center-to-center)

Updated: CLAUDE.md, hardware_constants.md, firmware/esp32/src/main.cpp,
docs/architecture/build_plan.md, src/robot_description/urdf/base.xacro
(base.xacro also has measured chassis dims: 240×203×51 mm)

Co-Authored-By: Claude Sonnet 4.6 <noreply@anthropic.com>

File: src/robot_description/urdf/base.xacro (robot description, xacro)
@@ -1,12 +1,12 @@
 <?xml version="1.0"?>
 <robot xmlns:xacro="http://www.ros.org/wiki/xacro">
+  <!-- Chassis estimates — measure and replace before Phase 3 EKF bringup -->
+  <xacro:property name="chassis_l" value="0.24"/>
+  <xacro:property name="chassis_w" value="0.203"/>
+  <xacro:property name="chassis_h" value="0.051"/>
   <!-- Validated hardware values — do not change without updating CLAUDE.md -->
-  <xacro:property name="wheel_radius" value="0.034"/>
-  <xacro:property name="wheel_width"  value="0.025"/>
-  <xacro:property name="wheel_sep"    value="0.179"/>
-  <!-- Chassis estimates — measure and replace before Phase 3 EKF bringup -->
-  <xacro:property name="chassis_l" value="0.200"/>
-  <xacro:property name="chassis_w" value="0.180"/>
-  <xacro:property name="chassis_h" value="0.100"/>
+  <xacro:property name="wheel_radius" value="0.033"/>
+  <xacro:property name="wheel_width"  value="0.026"/>
+  <xacro:property name="wheel_sep"    value="0.177"/>
   <!-- Inertia helpers -->
   <xacro:macro name="box_inertia" params="m l w h">

Commit message: Upgrade to 4-wheel skid steer + Cytron MDD10A motor driver
Hardware change:
- TB6612FNG (2-channel, 3A) → Cytron MDD10A (2-channel, 10A)
- 2-wheel diff drive → 4-wheel skid steer (2 JGA25-371 per side)

GPIO reassignment (10-13, frees 14-15):
- GPIO 10: PWM_R → MDD10A Ch1
- GPIO 11: DIR_R → MDD10A Ch1
- GPIO 12: PWM_L → MDD10A Ch2
- GPIO 13: DIR_L → MDD10A Ch2

Firmware: motors.h/cpp rewritten for PWM+DIR interface (simpler than TB6612
IN1/IN2 dual-direction pins). Same LEDC setup, same max speed constants.

URDF: base.xacro now has 4 wheel joints (front/rear × left/right).
Wheelbase placeholder 0.18 m — update when chassis arrives.

Updated: CLAUDE.md, hardware_constants.md, motors.h, motors.cpp,
base.xacro, robot_description/README.md

Co-Authored-By: Claude Sonnet 4.6 <noreply@anthropic.com>

File: src/robot_description/urdf/base.xacro (robot description, xacro)
@@ -1,12 +1,14 @@
 <?xml version="1.0"?>
 <robot xmlns:xacro="http://www.ros.org/wiki/xacro">
-  <!-- Chassis estimates — measure and replace before Phase 3 EKF bringup -->
-  <xacro:property name="chassis_l" value="0.24"/>
-  <xacro:property name="chassis_w" value="0.203"/>
-  <xacro:property name="chassis_h" value="0.051"/>
   <!-- Validated hardware values — do not change without updating CLAUDE.md -->
   <xacro:property name="wheel_radius" value="0.033"/>
   <xacro:property name="wheel_width"  value="0.026"/>
   <xacro:property name="wheel_sep"    value="0.177"/>
+  <!-- Measured chassis dimensions -->
+  <xacro:property name="chassis_l" value="0.24"/>
+  <xacro:property name="chassis_w" value="0.203"/>
+  <xacro:property name="chassis_h" value="0.051"/>
+  <!-- Wheelbase (front-to-rear axle distance) — PLACEHOLDER, measure when chassis arrives -->
+  <xacro:property name="wheelbase"    value="0.18"/>
   <!-- Inertia helpers -->
   <xacro:macro name="box_inertia" params="m l w h">
@@ -28,6 +30,6 @@
     </inertial>
   </xacro:macro>
-  <!-- Wheel macro — joint origin rpy="-pi/2 0 0" rotates cylinder z-axis onto parent y-axis -->
-  <xacro:macro name="wheel" params="name y_offset">
+  <!-- Wheel macro — joint origin rpy="-pi/2 0 0" aligns cylinder z-axis with parent y-axis -->
+  <xacro:macro name="wheel" params="name x_offset y_offset">
     <link name="${name}">
       <visual>
@@ -43,9 +45,9 @@
       <parent link="base_link"/>
       <child link="${name}"/>
-      <origin xyz="0 ${y_offset} 0" rpy="${-pi/2} 0 0"/>
+      <origin xyz="${x_offset} ${y_offset} 0" rpy="${-pi/2} 0 0"/>
       <axis xyz="0 0 1"/>
     </joint>
   </xacro:macro>
-  <!-- Base chassis — origin at wheel axle height, centered between wheels -->
+  <!-- Base chassis — origin at wheel axle height, centered between all four wheels -->
   <link name="base_link">
     <visual>
@@ -56,7 +58,10 @@
       <geometry><box size="${chassis_l} ${chassis_w} ${chassis_h}"/></geometry>
     </collision>
-    <xacro:box_inertia m="1.5" l="${chassis_l}" w="${chassis_w}" h="${chassis_h}"/>
+    <xacro:box_inertia m="2.5" l="${chassis_l}" w="${chassis_w}" h="${chassis_h}"/>
   </link>
-  <xacro:wheel name="left_wheel"  y_offset=" ${wheel_sep/2}"/>
-  <xacro:wheel name="right_wheel" y_offset="-${wheel_sep/2}"/>
+  <!-- Four wheels: front/rear × left/right -->
+  <xacro:wheel name="front_left_wheel"  x_offset=" ${wheelbase/2}" y_offset=" ${wheel_sep/2}"/>
+  <xacro:wheel name="front_right_wheel" x_offset=" ${wheelbase/2}" y_offset="-${wheel_sep/2}"/>
+  <xacro:wheel name="rear_left_wheel"   x_offset="-${wheelbase/2}" y_offset=" ${wheel_sep/2}"/>
+  <xacro:wheel name="rear_right_wheel"  x_offset="-${wheelbase/2}" y_offset="-${wheel_sep/2}"/>
 </robot>

Commit message: Update wheel radius to precise measured value (68.27mm)
wheel_radius: 0.033 → 0.03414 m (68.27mm diameter, caliper measurement)

Updated: CLAUDE.md, hardware_constants.md, firmware/esp32/src/main.cpp,
src/robot_description/urdf/base.xacro

Co-Authored-By: Claude Sonnet 4.6 <noreply@anthropic.com>

File: src/robot_description/urdf/base.xacro (robot description, xacro)
@@ -2,5 +2,5 @@
 <robot xmlns:xacro="http://www.ros.org/wiki/xacro">
   <!-- Validated hardware values — do not change without updating CLAUDE.md -->
-  <xacro:property name="wheel_radius" value="0.033"/>
+  <xacro:property name="wheel_radius" value="0.03414"/>
   <xacro:property name="wheel_width"  value="0.026"/>
   <xacro:property name="wheel_sep"    value="0.177"/>

Commit message: Update URDF chassis z-offset from measured bracket geometry
bracket_offset = 23mm: motor shaft sits 23mm below chassis plate bottom.
Chassis box visual/collision now correctly offset above wheel axle origin.
Ground clearance = 34.14mm (wheel_radius) - 23mm (bracket) = 11.14mm.

Co-Authored-By: Claude Sonnet 4.6 <noreply@anthropic.com>

File: src/robot_description/urdf/base.xacro (robot description, xacro)
@@ -10,5 +10,8 @@
   <xacro:property name="chassis_h" value="0.051"/>
   <!-- Wheelbase (front-to-rear axle distance) — PLACEHOLDER, measure when chassis arrives -->
-  <xacro:property name="wheelbase"    value="0.18"/>
+  <xacro:property name="wheelbase"      value="0.18"/>
+  <!-- Measured: motor shaft sits 23mm below chassis plate bottom surface.
+       Ground clearance = wheel_radius - bracket_offset = 34.14 - 23 = 11.14mm -->
+  <xacro:property name="bracket_offset" value="0.023"/>
   <!-- Inertia helpers -->
   <xacro:macro name="box_inertia" params="m l w h">
@@ -49,11 +52,14 @@
     </joint>
   </xacro:macro>
-  <!-- Base chassis — origin at wheel axle height, centered between all four wheels -->
+  <!-- Base chassis — origin at wheel axle height, centered between all four wheels.
+       Chassis bottom face is bracket_offset above the axle, so box center is offset in z. -->
   <link name="base_link">
     <visual>
+      <origin xyz="0 0 ${bracket_offset + chassis_h/2}" rpy="0 0 0"/>
       <geometry><box size="${chassis_l} ${chassis_w} ${chassis_h}"/></geometry>
       <material name="grey"/>
     </visual>
     <collision>
+      <origin xyz="0 0 ${bracket_offset + chassis_h/2}" rpy="0 0 0"/>
       <geometry><box size="${chassis_l} ${chassis_w} ${chassis_h}"/></geometry>
     </collision>

Commit message: fix(firmware): correct PID gains and deadband floor for 6.5 rad/s max speed
- MOTOR_MAX_RAD_S: 13.0 → 6.5 (measured max was 0.218 m/s, not 0.427)
- KP: 2.8 → 1.4, KI: 0.76 → 0.38 (rescaled from articubot_one gains)
- Fix deadband floor: only apply in direction of target; old code snapped
  small reverse corrections to -MOTOR_MIN_DUTY causing sustained oscillation

feat(urdf): Phase 2 TF tree complete and validated

- Add base_footprint root link (required by Nav2; eliminates KDL inertia warning)
- Fix joint_state_publisher: remove source_list: [] (Jazzy rclpy rejects
  empty-list params with unknown type); pass xacro file as positional arg
- All 9 frames connected: base_footprint → base_link → 4 wheels + laser +
  imu_link + camera_link → camera_depth_frame
- tf2_echo base_link laser returns correct static transform [0, 0, 0.18]

Co-Authored-By: Claude Sonnet 4.6 <noreply@anthropic.com>

File: src/robot_description/urdf/base.xacro (robot description, xacro)
@@ -52,4 +52,12 @@
     </joint>
   </xacro:macro>
+  <!-- base_footprint: ground-plane projection of base_link — required by Nav2 and robot_localization.
+       No geometry; KDL complains if the root link has inertia, so this link carries none. -->
+  <link name="base_footprint"/>
+  <joint name="base_footprint_joint" type="fixed">
+    <parent link="base_footprint"/>
+    <child link="base_link"/>
+    <origin xyz="0 0 0" rpy="0 0 0"/>
+  </joint>
   <!-- Base chassis — origin at wheel axle height, centered between all four wheels.
        Chassis bottom face is bracket_offset above the axle, so box center is offset in z. -->
